Commit message: use package:// for file path in xacro

File: urdf/xacro/thing_no_wheels.urdf.xacro (robot description, xacro)
@@ -58,5 +58,5 @@
     <visual>
       <geometry>
-        <mesh filename="file://$(find mobile_manipulation_central)/meshes/ridgeback/body.stl"/>
+        <mesh filename="package://mobile_manipulation_central/meshes/ridgeback/body.stl"/>
       </geometry>
       <material name="black"/>
@@ -65,5 +65,5 @@
       <origin xyz="0 0 0"/>
       <geometry>
-        <mesh filename="file://$(find mobile_manipulation_central)/meshes/ridgeback/body-collision.stl"/>
+        <mesh filename="package://mobile_manipulation_central/meshes/ridgeback/body-collision.stl"/>
       </geometry>
     </collision>
@@ -89,5 +89,5 @@
       <origin rpy="0 0 3.14159265359" xyz="0 0 0"/>
       <geometry>
-        <mesh filename="file://$(find mobile_manipulation_central)/meshes/ridgeback/side-cover.stl"/>
+        <mesh filename="package://mobile_manipulation_central/meshes/ridgeback/side-cover.stl"/>
       </geometry>
       <material name="yellow"/>
@@ -98,5 +98,5 @@
       <origin rpy="0 0 0" xyz="0 0 0"/>
       <geometry>
-        <mesh filename="file://$(find mobile_manipulation_central)/meshes/ridgeback/side-cover.stl"/>
+        <mesh filename="package://mobile_manipulation_central/meshes/ridgeback/side-cover.stl"/>
       </geometry>
       <material name="yellow"/>
@@ -112,5 +112,5 @@
       <origin rpy="0 0 0" xyz="0 0 0"/>
       <geometry>
-        <mesh filename="file://$(find mobile_manipulation_central)/meshes/ridgeback/end-cover.stl"/>
+        <mesh filename="package://mobile_manipulation_central/meshes/ridgeback/end-cover.stl"/>
       </geometry>
       <material name="black"/>
@@ -126,5 +126,5 @@
       <origin rpy="0 0 3.14159265359" xyz="0 0 0"/>
       <geometry>
-        <mesh filename="file://$(find mobile_manipulation_central)/meshes/ridgeback/end-cover.stl"/>
+        <mesh filename="package://mobile_manipulation_central/meshes/ridgeback/end-cover.stl"/>
       </geometry>
       <material name="black"/>
@@ -145,5 +145,5 @@
       <origin rpy="0 0 0" xyz="0 0 0"/>
       <geometry>
-        <mesh filename="file://$(find mobile_manipulation_central)/meshes/ridgeback/lights.stl"/>
+        <mesh filename="package://mobile_manipulation_central/meshes/ridgeback/lights.stl"/>
       </geometry>
       <material name="white"/>
@@ -154,5 +154,5 @@
       <origin rpy="0 0 3.14159265359" xyz="0 0 0"/>
       <geometry>
-        <mesh filename="file://$(find mobile_manipulation_central)/meshes/ridgeback/lights.stl"/>
+        <mesh filename="package://mobile_manipulation_central/meshes/ridgeback/lights.stl"/>
       </geometry>
       <material name="red"/>
@@ -168,5 +168,5 @@
       <origin rpy="0 0 0" xyz="0 0 0"/>
       <geometry>
-        <mesh filename="file://$(find mobile_manipulation_central)/meshes/ridgeback/top.stl"/>
+        <mesh filename="package://mobile_manipulation_central/meshes/ridgeback/top.stl"/>
       </geometry>
       <material name="black"/>
@@ -175,5 +175,5 @@
       <origin rpy="0 0 0" xyz="0 0 0"/>
       <geometry>
-        <mesh filename="file://$(find mobile_manipulation_central)/meshes/ridgeback/top.stl"/>
+        <mesh filename="package://mobile_manipulation_central/meshes/ridgeback/top.stl"/>
       </geometry>
     </collision>
@@ -182,5 +182,5 @@
     <visual>
       <geometry>
-        <mesh filename="file://$(find mobile_manipulation_central)/meshes/tor11_mech.dae"/>
+        <mesh filename="package://mobile_manipulation_central/meshes/tor11_mech.dae"/>
       </geometry>
       <material name="LightGrey">
