Commit message: Fuse Ridgeback odom velocity with gated Vicon pose for hardware teleop/MPC.
Replace the TF+odom estimator with rate-limited Vicon corrections and
innovation gates so /ridgeback/joint_states velocity stays odom-derived.
Update lab remaps (ThingBase_Fed), Vicon host, launch defaults, and docs;
add bag validation; shorten the gripper pole so angled trays do not pierce.

File: urdf/xacro/thing.urdf.xacro (robot description, xacro)
@@ -3,6 +3,6 @@
   <xacro:include filename="ridgeback_wheels.urdf.xacro" />
   <xacro:include filename="thing_no_wheels.urdf.xacro" />
-  <xacro:include filename="$(find mmseq_assets)/thing/xacro/collision.urdf.xacro" />
-  <xacro:include filename="$(find mmseq_assets)/thing/xacro/end_effector_fingers.urdf.xacro" />
+  <!-- <xacro:include filename="$(find mmseq_assets)/thing/xacro/collision.urdf.xacro" /> -->
+  <!-- <xacro:include filename="$(find mmseq_assets)/thing/xacro/end_effector_fingers.urdf.xacro" /> -->
 <!--  <xacro:include filename="$(find mmseq_assets)/thing/xacro/end_effector_box.urdf.xacro" />-->
 </robot>

File: urdf/xacro/thing_no_wheels.urdf.xacro (robot description, xacro)
@@ -211,15 +211,15 @@
   <link name="gripper">
     <visual>
-      <!-- start halfway along the cylinder -->
-      <origin rpy="0 0 0" xyz="0 0 0.145"/>
-      <geometry>
-        <cylinder length="0.290" radius="0.01"/>
+      <!-- Tip stops at the angled tray underside so the pole does not pierce the disk. -->
+      <origin rpy="0 0 0" xyz="0 0 0.115"/>
+      <geometry>
+        <cylinder length="0.230" radius="0.01"/>
       </geometry>
       <material name="black"/>
     </visual>
     <collision>
-      <origin rpy="0 0 0" xyz="0 0 0.145"/>
-      <geometry>
-        <cylinder length="0.290" radius="0.01"/>
+      <origin rpy="0 0 0" xyz="0 0 0.115"/>
+      <geometry>
+        <cylinder length="0.230" radius="0.01"/>
       </geometry>
     </collision>
